File: hardware/phantasm/phantasm.kicad_sch (KiCad schematic)
At the start: 29 parts, among them J1 +5V IN ~1A, J2 LED sig DI/CI/SIG_GND, J3A SYNC in, J3B SYNC out, J4 debug, U1 74AHCT125

Commit message: updated PCB gen
Parts:
- F1: value 0.75A -> 0.5A
Changed lines of the file:
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@@
 			(effects (font (size 1.27 1.27)))
 		)
-		(property "Value" "0.75A"
+		(property "Value" "0.5A"
 			(at 40.64 66.04 0)
 			(effects (font (size 1.27 1.27)))
