File: hardware/phantasm/phantasm.kicad_sch (KiCad schematic)
At the start: 28 parts, among them J1 +5V IN ~1A, J2 LED sig DI/CI/SIG_GND, J3A SYNC in, J3B SYNC out, J4 debug, U1 74AHCT125

Commit message: pcb: align schematic assembly metadata with routed board (finding 16)
Parts:
- C_IN, J1, J2, J3A, J3B, J4: now left out of the parts list
- U_MCU: footprint (none) -> phantasm:Teensy4.0; now left out of the parts list
Changed lines of the file:
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@@
 		(unit 1)
 		(exclude_from_sim no)
-		(in_bom yes)
+		(in_bom no)
 		(on_board yes)
 		(dnp no)
@@
 		(unit 1)
 		(exclude_from_sim no)
-		(in_bom yes)
+		(in_bom no)
 		(on_board yes)
 		(dnp no)
@@
 		(unit 1)
 		(exclude_from_sim no)
-		(in_bom yes)
+		(in_bom no)
 		(on_board yes)
 		(dnp no)
@@
 			(effects (font (size 1.27 1.27)))
 		)
-		(property "Footprint" ""
+		(property "Footprint" "phantasm:Teensy4.0"
 			(at 60.96 172.72 0)
 			(effects (font (size 1.27 1.27)) (hide yes))
@@
 		(unit 1)
 		(exclude_from_sim no)
-		(in_bom yes)
+		(in_bom no)
 		(on_board yes)
 		(dnp no)
@@
 		(unit 1)
 		(exclude_from_sim no)
-		(in_bom yes)
+		(in_bom no)
 		(on_board yes)
 		(dnp no)
@@
 		(unit 1)
 		(exclude_from_sim no)
-		(in_bom yes)
+		(in_bom no)
 		(on_board yes)
 		(dnp no)
@@
 		(unit 1)
 		(exclude_from_sim no)
-		(in_bom yes)
-		(on_board yes)
-		(dnp no)
+		(in_bom no)
+		(on_board yes)
+		(dnp no)
