File: hardware/phantasm/phantasm.kicad_pcb (KiCad board)
At the start: 4 copper layers, 58.3 x 32 mm, 32 parts, among them J1 +5V IN ~1A, J2 LED sig DI/CI/SIG_GND, J3A SYNC in, J3B SYNC out, J4 debug, U1 74AHCT125

Commit message: phantasm: remove bottom trace acute corner
Routing:
- net /MASTER_EN: track 42.3 -> 41.2 mm, vias 4 -> 5
- net GND: vias 87 -> 86
Changed lines of the file:
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@@
-	)
-	(via
-		(at 23.984134 22.910562)
-		(size 0.45)
-		(drill 0.2)
-		(layers "F.Cu" "B.Cu")
-		(net "GND")
 	)
 	(via
@@
 	)
 	(via
+		(at 23.984134 22.910562)
+		(size 0.45)
+		(drill 0.2)
+		(layers "F.Cu" "B.Cu")
+		(net "/MASTER_EN")
+	)
+	(via
 		(at 16.340002 22.506187)
 		(size 0.45)
@@
 	)
 	(segment
-		(start 24.544 24)
+		(start 23.544 23.506)
 		(end 18.018351 23.506)
 		(width 0.13)
@@
 	(segment
 		(start 24.544 22.506)
-		(end 24.544 24)
-		(width 0.13)
-		(layer "B.Cu")
+		(end 23.544 23.506)
+		(width 0.13)
+		(layer "B.Cu")
