File: hardware/phantasm/phantasm.kicad_pcb (KiCad board)
At the start: 4 copper layers, 58.3 x 32 mm, 32 parts, among them J1 +5V IN ~1A, J2 LED sig DI/CI/SIG_GND, J3A SYNC in, J3B SYNC out, J4 debug, U1 74AHCT125

Commit message: pcb: restore JP_ID2 silkscreen (finding 65)
Other:
- board text added: "N8 ID2 OPEN=0-3 GND=4-7; M=OPEN; SHLD=M"
- board text removed: "MASTER = ALL ID OPEN SHLD = MASTER ONLY"
Changed lines of the file:
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@@
 				(type solid)
 			)
-			(layer "F.Fab")
+			(layer "F.SilkS")
 		)
 		(fp_line
@@
 				(type solid)
 			)
-			(layer "F.Fab")
+			(layer "F.SilkS")
 		)
 		(fp_line
@@
 				(type solid)
 			)
-			(layer "F.Fab")
+			(layer "F.SilkS")
 		)
 		(fp_line
@@
 				(type solid)
 			)
-			(layer "F.Fab")
+			(layer "F.SilkS")
 		)
 		(fp_arc
@@
 				(type solid)
 			)
-			(layer "F.Fab")
+			(layer "F.SilkS")
 		)
 		(fp_arc
@@
 				(type solid)
 			)
-			(layer "F.Fab")
+			(layer "F.SilkS")
 		)
 		(fp_arc
@@
 				(type solid)
 			)
-			(layer "F.Fab")
+			(layer "F.SilkS")
 		)
 		(fp_arc
@@
 				(type solid)
 			)
-			(layer "F.Fab")
+			(layer "F.SilkS")
 		)
 		(pad "1" smd custom
@@
 		)
 	)
-	(gr_text "MASTER = ALL ID OPEN   SHLD = MASTER ONLY"
+	(gr_text "N8 ID2 OPEN=0-3 GND=4-7; M=OPEN; SHLD=M"
 		(at 29.14 17 0)
 		(layer "B.SilkS")
