File: hardware/phantasm/phantasm.kicad_pcb (KiCad board)
At the start: 4 copper layers, 58.3 x 32 mm, 32 parts, among them J1 +5V IN ~1A, J2 LED sig DI/CI/SIG_GND, J3A SYNC in, J3B SYNC out, J4 debug, U1 74AHCT125

Commit message: hardware: raise sync TVS standoff above the drive rail (finding 317)
Parts:
- D_BUS: value CDSOD323-T05L -> CDSOD323-T08L
Changed lines of the file:
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@@
 			)
 		)
-		(property "Value" "CDSOD323-T05L"
+		(property "Value" "CDSOD323-T08L"
 			(at 0.1 1.9 0)
 			(layer "F.Fab")

Commit message: hardware: place the strip return between data and clock (finding 318)
Parts:
- J2: value LED sig DI/CI/SIG_GND -> LED sig DI/SIG_GND/CI
Connections:
- J2 pad 2: /CLK -> GND
- J2 pad 3: GND -> /CLK
Routing:
- net /CLK: track 21.6 -> 20.5 mm
Changed lines of the file:
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@@
 			)
 		)
-		(property "Value" "LED sig DI/CI/SIG_GND"
+		(property "Value" "LED sig DI/SIG_GND/CI"
 			(at 0 7.46 0)
 			(layer "F.Fab")
@@
 			(layers "*.Cu" "*.Mask")
 			(remove_unused_layers no)
-			(net "/CLK")
+			(net "GND")
 		)
 		(pad "3" thru_hole circle
@@
 			(layers "*.Cu" "*.Mask")
 			(remove_unused_layers no)
-			(net "GND")
+			(net "/CLK")
 		)
 		(embedded_fonts no)
@@
 		)
 	)
-	(gr_text "C"
+	(gr_text "G"
 		(at 52 5.31 0)
 		(layer "F.SilkS")
@@
 		)
 	)
-	(gr_text "G"
+	(gr_text "C"
 		(at 52 7.85 0)
 		(layer "F.SilkS")
@@
 	)
 	(segment
-		(start 48.986781 6.123219)
-		(end 49.497575 5.612425)
+		(start 46.875648 10.774352)
+		(end 49.497575 8.152425)
 		(width 0.13)
 		(layer "B.Cu")
@@
 	)
 	(segment
-		(start 49.497575 5.612425)
-		(end 49.8 5.31)
+		(start 49.497575 8.152425)
+		(end 49.8 7.85)
 		(width 0.13)
 		(layer "B.Cu")
@@
 	(segment
 		(start 44.335648 10.774352)
-		(end 48.986781 6.123219)
+		(end 46.875648 10.774352)
 		(width 0.13)
 		(layer "B.Cu")
