File: hardware/phantasm/1.2/phantasm.kicad_sch (KiCad schematic)
At the start: 29 parts, among them J1 +5V IN ~1A, J2 LED sig DI/CI/SIG_GND, J3A SYNC in, J3B SYNC out, J4 debug, U1 74AHCT125

Commit message: pcb: organize revision projects and complete Teensy pin parity
Parts:
- removed D_BUS: TVS, Diode_SMD:D_SOD-323, symbol Device:D_TVS
- removed R_ID0: 10k DNP, Resistor_SMD:R_0603_1608Metric, symbol Device:R
- added D_BUS: CDSOD323-T08L, Diode_SMD:D_SOD-323, symbol Device:D_Zener
- added R_TX: 10k, Resistor_SMD:R_0603_1608Metric, symbol Device:R
- C_IN, J4, JP_ID0, JP_ID1, JP_ID2, JP_SHLD: now left out of the parts list
- J1: value +5V IN ~1A -> TBC05-02-1-G-G +5V IN ~1A; footprint Connector_PinHeader_2.54mm:PinHeader_1x02_P2.54mm_Vertical -> phantasm:TerminalBlock_GCT_TBC05-02-1-G-G; now left out of the parts list
- J2: value LED sig DI/CI/SIG_GND -> TBC05-03-1-G-G LED DI/SIG_GND/CI; footprint Connector_PinHeader_2.54mm:PinHeader_1x03_P2.54mm_Vertical -> phantasm:TerminalBlock_GCT_TBC05-03-1-G-G; now left out of the parts list
- J3A: value SYNC in -> TBC05-03-1-G-G SYNC in; footprint Connector_PinHeader_2.54mm:PinHeader_1x03_P2.54mm_Vertical -> phantasm:TerminalBlock_GCT_TBC05-03-1-G-G; now left out of the parts list
- J3B: value SYNC out -> TBC05-03-1-G-G SYNC out; footprint Connector_PinHeader_2.54mm:PinHeader_1x03_P2.54mm_Vertical -> phantasm:TerminalBlock_GCT_TBC05-03-1-G-G; now left out of the parts list
- R1, R2, R_PD: footprint Resistor_SMD:R_0603_1608Metric -> Resistor_SMD:R_0603_1608Metric_Pad0.98x0.95mm_HandSolder
- R_S: footprint Resistor_SMD:R_0805_2012Metric -> Resistor_SMD:R_0805_2012Metric_Pad1.20x1.40mm_HandSolder
- U_MCU: footprint (none) -> phantasm:Teensy4.0; now left out of the parts list
Connections:
- net CLK: now also J2.3 (Pin_3); no longer J2.2 (Pin_2)
- net FRAME_SYNC: no longer U1.9
- net GND: now also J2.2 (Pin_2), D_BUS.2 (A), R_TX.2; no longer J2.3 (Pin_3)
- net SYNC_BUS: now also D_BUS.1 (K)
- new net SYNC_TX: R_TX.1, U1.9, U_MCU.4 (D4)
- no-connect marks 0 -> 15

Commit message: pcb: remove unused rev 1.2 debug header and serial connection
Parts:
- removed J4: debug, Connector_PinHeader_2.54mm:PinHeader_1x04_P2.54mm_Vertical, symbol Connector_Generic:Conn_01x04
Connections:
- net SERIAL1_TX: no longer names the net of U_MCU.1 (D1/TX1)
- no-connect marks 15 -> 16
Other:
- note added: "ID STRAPS / MASTER_EN PULL-UP"
- note removed: "ID STRAPS / MASTER_EN PULL-UP / DEBUG"
Changed lines of the file:
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@@
 		(color 0 0 0 0)
 	)
+	(no_connect (at 41.91 170.18))
 	(no_connect (at 80.01 134.62))
 	(no_connect (at 80.01 137.16))
@@
 	)
 	(wire
-		(pts (xy 41.91 170.18) (xy 38.1 170.18))
-		(stroke (width 0) (type default))
-	)
-	(wire
 		(pts (xy 144.78 137.16) (xy 140.97 137.16))
 		(stroke (width 0) (type default))
@@
 	(wire
 		(pts (xy 182.88 274.32) (xy 185.42 274.32))
-		(stroke (width 0) (type default))
-	)
-	(wire
-		(pts (xy 33.02 264.16) (xy 30.48 264.16))
-		(stroke (width 0) (type default))
-	)
-	(wire
-		(pts (xy 33.02 266.7) (xy 30.48 266.7))
-		(stroke (width 0) (type default))
-	)
-	(wire
-		(pts (xy 33.02 269.24) (xy 29.21 269.24))
-		(stroke (width 0) (type default))
-	)
-	(wire
-		(pts (xy 33.02 271.78) (xy 29.21 271.78))
 		(stroke (width 0) (type default))
 	)
@@
 		(effects (font (size 1.27 1.27)) (justify left bottom))
 	)
-	(label "SERIAL1_TX"
-		(at 38.1 170.18 0)
-		(effects (font (size 1.27 1.27)) (justify left bottom))
-	)
 	(label "DATA_IN"
 		(at 140.97 137.16 0)
@@
 	(label "ID2"
 		(at 168.91 274.32 0)
-		(effects (font (size 1.27 1.27)) (justify left bottom))
-	)
-	(label "MASTER_EN"
-		(at 29.21 269.24 0)
-		(effects (font (size 1.27 1.27)) (justify left bottom))
-	)
-	(label "SERIAL1_TX"
-		(at 29.21 271.78 0)
 		(effects (font (size 1.27 1.27)) (justify left bottom))
 	)
@@
 		(effects (font (size 2.2 2.2) (bold yes)) (justify left bottom))
 	)
-	(text "ID STRAPS / MASTER_EN PULL-UP / DEBUG"
+	(text "ID STRAPS / MASTER_EN PULL-UP"
 		(at 25 245 0)
 		(effects (font (size 2.2 2.2) (bold yes)) (justify left bottom))
@@
 	)
 	(symbol
-		(lib_id "Connector_Generic:Conn_01x04")
-		(at 38.1 266.7 0)
-		(unit 1)
-		(exclude_from_sim no)
-		(in_bom no)
-		(on_board yes)
-		(dnp no)
-		(property "Reference" "J4"
-			(at 38.1 261.62 0)
-			(effects (font (size 1.27 1.27)))
-		)
-		(property "Value" "debug"
-			(at 38.1 271.78 0)
-			(effects (font (size 1.27 1.27)))
-		)
-		(property "Footprint" "Connector_PinHeader_2.54mm:PinHeader_1x04_P2.54mm_Vertical"
-			(at 38.1 274.32 0)
-			(effects (font (size 1.27 1.27)) (hide yes))
-		)
-		(property "Datasheet" ""
-			(at 38.1 266.7 0)
-			(effects (font (size 1.27 1.27)) (hide yes))
-		)
-		(pin "1")
-		(pin "2")
-		(pin "3")
-		(pin "4")
-		(instances
-			(project "phantasm"
-				(path "/0060d4b9-1e71-57bc-bde8-9bde7b0cc02a"
-					(reference "J4") (unit 1)
-				)
-			)
-		)
-	)
-	(symbol
-		(lib_id "power:+3V3")
-		(at 30.48 264.16 0)
-		(unit 1)
-		(exclude_from_sim no)
-		(in_bom yes)
-		(on_board yes)
-		(dnp no)
-		(property "Reference" "#PWR25"
-			(at 30.48 259.08 0)
-			(effects (font (size 1.27 1.27)))
-		)
-		(property "Value" "+3V3"
-			(at 30.48 269.24 0)
-			(effects (font (size 1.27 1.27)))
-		)
-		(property "Footprint" ""
-			(at 30.48 271.78 0)
-			(effects (font (size 1.27 1.27)) (hide yes))
-		)
-		(property "Datasheet" ""
-			(at 30.48 264.16 0)
-			(effects (font (size 1.27 1.27)) (hide yes))
-		)
-		(pin "1")
-		(instances
-			(project "phantasm"
-				(path "/0060d4b9-1e71-57bc-bde8-9bde7b0cc02a"
-					(reference "#PWR25") (unit 1)
-				)
-			)
-		)
-	)
-	(symbol
-		(lib_id "power:GND")
-		(at 30.48 266.7 0)
-		(unit 1)
-		(exclude_from_sim no)
-		(in_bom yes)
-		(on_board yes)
-		(dnp no)
-		(property "Reference" "#PWR26"
-			(at 30.48 261.62 0)
-			(effects (font (size 1.27 1.27)))
-		)
-		(property "Value" "GND"
-			(at 30.48 271.78 0)
-			(effects (font (size 1.27 1.27)))
-		)
-		(property "Footprint" ""
-			(at 30.48 274.32 0)
-			(effects (font (size 1.27 1.27)) (hide yes))
-		)
-		(property "Datasheet" ""
-			(at 30.48 266.7 0)
-			(effects (font (size 1.27 1.27)) (hide yes))
-		)
-		(pin "1")
-		(instances
-			(project "phantasm"
-				(path "/0060d4b9-1e71-57bc-bde8-9bde7b0cc02a"
-					(reference "#PWR26") (unit 1)
-				)
-			)
-		)
-	)
-	(symbol
 		(lib_id "phantasm:+5V_RAW")
 		(at 246.38 274.32 0)
@@
 		(on_board yes)
 		(dnp no)
-		(property "Reference" "#PWR27"
+		(property "Reference" "#PWR25"
 			(at 246.38 269.24 0)
 			(effects (font (size 1.27 1.27)))
@@
 			(project "phantasm"
 				(path "/0060d4b9-1e71-57bc-bde8-9bde7b0cc02a"
-					(reference "#PWR27") (unit 1)
+					(reference "#PWR25") (unit 1)
 				)
 			)
@@
 		(on_board yes)
 		(dnp no)
-		(property "Reference" "#PWR28"
+		(property "Reference" "#PWR26"
 			(at 284.48 269.24 0)
 			(effects (font (size 1.27 1.27)))
@@
 			(project "phantasm"
 				(path "/0060d4b9-1e71-57bc-bde8-9bde7b0cc02a"
-					(reference "#PWR28") (unit 1)
+					(reference "#PWR26") (unit 1)
 				)
 			)
@@
 		(on_board yes)
 		(dnp no)
-		(property "Reference" "#PWR29"
+		(property "Reference" "#PWR27"
 			(at 317.5 269.24 0)
 			(effects (font (size 1.27 1.27)))
@@
 			(project "phantasm"
 				(path "/0060d4b9-1e71-57bc-bde8-9bde7b0cc02a"
-					(reference "#PWR29") (unit 1)
-				)
-			)
+					(reference "#PWR27") (unit 1)
+				)
+			)

Commit message: pcb: clarify bypass parents and enforce upload via minimum
Parts:
- removed D_BUS: CDSOD323-T08L, Diode_SMD:D_SOD-323, symbol Device:D_Zener
- removed J2: TBC05-03-1-G-G LED DI/SIG_GND/CI, phantasm:TerminalBlock_GCT_TBC05-03-1-G-G, symbol Connector_Generic:Conn_01x03
- removed JP_SHLD: shield gnd (master only), Jumper:SolderJumper-2_P1.3mm_Open_RoundedPad1.0x1.5mm, symbol Jumper:SolderJumper_2_Open
- removed U_MCU: Teensy4.0, phantasm:Teensy4.0, symbol phantasm:Teensy4.0
- added C_DEC2: 0.1uF, Capacitor_SMD:C_0603_1608Metric, symbol Device:C
- added C_SYNC: 220pF, Capacitor_SMD:C_0603_1608Metric, symbol Device:C
- added J3A: TBC05-03-1-G-G SYNC in, phantasm:TerminalBlock_GCT_TBC05-03-1-G-G, symbol Connector_Generic:Conn_01x03
- added JP_ID2: ID2->GND (N=8), Jumper:SolderJumper-2_P1.3mm_Open_RoundedPad1.0x1.5mm, symbol Jumper:SolderJumper_2_Open
- D_BUS: renamed from J3A; value TBC05-03-1-G-G SYNC in -> CDSOD323-T08L; footprint phantasm:TerminalBlock_GCT_TBC05-03-1-G-G -> Diode_SMD:D_SOD-323; symbol Connector_Generic:Conn_01x03 -> Device:D_Zener; now in the parts list
- J2: renamed from R1; value 10k -> TBC05-03-1-G-G LED DI/SIG_GND/CI; footprint Resistor_SMD:R_0603_1608Metric_Pad0.98x0.95mm_HandSolder -> phantasm:TerminalBlock_GCT_TBC05-03-1-G-G; symbol Device:R -> Connector_Generic:Conn_01x03; now left out of the parts list
- JP_ID0: renamed from JP_ID1; value ID1->GND -> ID0->GND
- JP_ID1: renamed from JP_ID2; value ID2->GND (N=8) -> ID1->GND
- JP_SHLD: renamed from R_MEN; value 10k -> shield gnd (master only); footprint Resistor_SMD:R_0603_1608Metric -> Jumper:SolderJumper-2_P1.3mm_Open_RoundedPad1.0x1.5mm; symbol Device:R -> Jumper:SolderJumper_2_Open; now left out of the parts list
- R1: renamed from C_SYNC; value 220pF -> 10k; footprint Capacitor_SMD:C_0603_1608Metric -> Resistor_SMD:R_0603_1608Metric_Pad0.98x0.95mm_HandSolder; symbol Device:C -> Device:R
- R_MEN: renamed from JP_ID0; value ID0->GND -> 10k; footprint Jumper:SolderJumper-2_P1.3mm_Open_RoundedPad1.0x1.5mm -> Resistor_SMD:R_0603_1608Metric; symbol Jumper:SolderJumper_2_Open -> Device:R; now in the parts list
- U_MCU: renamed from C_DEC2; value 0.1uF -> Teensy4.0; footprint Capacitor_SMD:C_0603_1608Metric -> phantasm:Teensy4.0; symbol Device:C -> phantasm:Teensy4.0; now left out of the parts list
Connections:
- net +3V3: now also R_MEN.1, U_MCU.3V3; no longer JP_SHLD.1
- net +5V_LOGIC: now also U_MCU.VIN, C_DEC2.1; no longer U_MCU.1
- net CLK: now also J2.3 (Pin_3)
- net CLK_IN: now also U_MCU.13 (D13/SCK)
- net DATA: now also J2.1 (Pin_1)
- net DATA_IN: now also U_MCU.11 (D11/MOSI)
- net FRAME_SYNC: now also R1.2, U_MCU.3 (D3), C_SYNC.1; no longer J2.2, R1.1
- net GND: now also J2.2 (Pin_2), JP_SHLD.2 (B), U_MCU.GND, C_DEC2.2, C_SYNC.2, J3A.2 (Pin_2), JP_ID2.2 (B); no longer R1.2, R_MEN.2 (B), U_MCU.2
- net ID0: now also JP_ID0.1 (A), U_MCU.21 (D21); no longer R_MEN.1 (A)
- net ID1: now also JP_ID1.1 (A), U_MCU.22 (D22); no longer JP_ID0.1 (A)
- net ID2: now also U_MCU.23 (D23), JP_ID2.1 (A); no longer JP_ID1.1 (A)
- net MASTER_EN: now also R_MEN.2, U_MCU.5 (D5); no longer JP_SHLD.2
- net SHIELD: now also JP_SHLD.1 (A), J3A.3 (Pin_3); no longer D_BUS.3 (Pin_3)
- net SYNC_BUS: now also R1.1, J3A.1 (Pin_1); no longer J2.1
- net SYNC_TX: now also U_MCU.4 (D4)
Other:
- moved on the sheet: JP_ID0, JP_ID1
