File: hardware/phantasm/1.3/phantasm.kicad_pcb (KiCad board)
At the start: 4 copper layers, 58.3 x 32 mm, 36 parts, among them J1 TBC05-02-1-G-G +5V IN ~1A, J2 TBC05-03-1-G-G LED DI/SIG_GND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, J3A TBC05-04-1-G-G SYNC in, J3B TBC05-04-1-G-G SYNC out, U1 74AHCT125

Commit message: pcb: label four-board ID roles explicitly (finding 11)
Other:
- board text added: "ID ID0 ID1 ROLE(N4)"
- board text removed: "ID ID0 ID1 ROLE"
Changed lines of the file:
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@@
 	(gr_text "SYNC IN" (at 46 6.5 90) (layer "B.SilkS") (effects (font (size 0.8 0.8) (thickness 0.15)) (justify mirror)))
 	(gr_text "SYNC OUT" (at 46 19.06 90) (layer "B.SilkS") (effects (font (size 0.8 0.8) (thickness 0.15)) (justify mirror)))
-	(gr_text "ID  ID0   ID1   ROLE" (at 25.5 7 0) (layer "B.SilkS") (effects (font (size 0.9 0.9) (thickness 0.15)) (justify mirror)))
+	(gr_text "ID  ID0   ID1   ROLE(N4)" (at 25.5 7 0) (layer "B.SilkS") (effects (font (size 0.9 0.9) (thickness 0.15)) (justify mirror)))
 	(gr_text "0   OPEN  OPEN  MASTER" (at 25.5 9 0) (layer "B.SilkS") (effects (font (size 0.9 0.9) (thickness 0.15)) (justify mirror)))
 	(gr_text "1   GND   OPEN  A-SOUTH" (at 25.5 11 0) (layer "B.SilkS") (effects (font (size 0.9 0.9) (thickness 0.15)) (justify mirror)))
